File: Hardware/matt_damon/matt_damon.kicad_pcb (KiCad board)
At the start: 2 copper layers, 52.3 x 46 mm, 20 parts, among them J1 ICSP, U1 ATtiny85V-10PU, X1 Badgelife_sao_connector_v169b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

Commit message: matt damon!
Parts:
- removed the G*** at (0.00, 0.00) (x6)
- added G*** (x6): LOGO, LOGO, F.Cu at (0.00, 0.00)
- D1, D4: value LED -> LED RED
- D2: value LED -> LED Orange
- D3: value LED -> LED Blue
- D5: value LED -> LED Yellow
- U1: footprint digikey-footprints:SOIC-8_W5.3mm -> Package_SO:SOIJ-8_5.3x5.3mm_P1.27mm
- moved R5 2.63 mm to (0.94, -23.9)
- moved U1 1.44 mm to (-6.21, -22.5)
Routing:
- net PB3: track 7.93 -> 9.79 mm
- net RST: track 15.8 -> 17.6 mm
- net Net-(D5-Pad2): track 4.45 -> 6.25 mm
- net SCK: track 17.8 -> 19.3 mm
- net MOSI: track 24.1 -> 25.0 mm
- net MISO: track 17.9 -> 18.8 mm
- net +3V3: track 6.21 -> 5.39 mm
Other:
- board text added: "JLCJLCJLCJLC"
