File: Hardware/matt_damon/matt_damon.sch (KiCad schematic (older format))
At the start: 14 parts, among them J1 ICSP, U1 ATtiny85V-10PU, X1 Badgelife_sao_connector_v169b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

Commit message: matt damon!
Parts:
- D1, D4: value LED -> LED RED
- D2: value LED -> LED Orange
- D3: value LED -> LED Blue
- D5: value LED -> LED Yellow
- U1: footprint digikey-footprints:SOIC-8_W5.3mm -> Package_SO:SOIJ-8_5.3x5.3mm_P1.27mm
Changed lines of the file:
@@
 F 0 "U1" H 3795 3021 50  0000 R CNN
 F 1 "ATtiny85V-10PU" H 3795 2930 50  0000 R CNN
-F 2 "digikey-footprints:SOIC-8_W5.3mm" H 4325 2975 50  0001 C CIN
+F 2 "Package_SO:SOIJ-8_5.3x5.3mm_P1.27mm" H 4325 2975 50  0001 C CIN
 F 3 "http://ww1.microchip.com/downloads/en/DeviceDoc/atmel-2586-avr-8-bit-microcontroller-attiny25-attiny45-attiny85_datasheet.pdf" H 4325 2975 50  0001 C CNN
 	1    4325 2975
@@
 NoConn ~ 5720 4875
 $Comp
-L Device:R R1
-U 1 1 5F1702EA
-P 3530 1265
-F 0 "R1" V 3323 1265 50  0000 C CNN
-F 1 "R" V 3414 1265 50  0000 C CNN
-F 2 "Resistor_SMD:R_0805_2012Metric_Pad1.15x1.40mm_HandSolder" V 3460 1265 50  0001 C CNN
-F 3 "~" H 3530 1265 50  0001 C CNN
-	1    3530 1265
-	0    1    1    0
-$EndComp
-$Comp
 L Device:LED D3
 U 1 1 5D7D1B19
 P 5750 1300
 F 0 "D3" H 5743 1516 50  0000 C CNN
-F 1 "LED" H 5743 1425 50  0000 C CNN
+F 1 "LED Blue" H 5743 1425 50  0000 C CNN
 F 2 "LED_SMD:LED_1206_3216Metric" H 5750 1300 50  0001 C CNN
 F 3 "~" H 5750 1300 50  0001 C CNN
@@
 P 7060 1310
 F 0 "D4" H 7053 1526 50  0000 C CNN
-F 1 "LED" H 7053 1435 50  0000 C CNN
+F 1 "LED RED" H 7053 1435 50  0000 C CNN
 F 2 "LED_SMD:LED_1206_3216Metric" H 7060 1310 50  0001 C CNN
 F 3 "~" H 7060 1310 50  0001 C CNN
@@
 P 4455 1305
 F 0 "D2" H 4448 1521 50  0000 C CNN
-F 1 "LED" H 4448 1430 50  0000 C CNN
+F 1 "LED Orange" H 4448 1430 50  0000 C CNN
 F 2 "LED_SMD:LED_1206_3216Metric" H 4455 1305 50  0001 C CNN
 F 3 "~" H 4455 1305 50  0001 C CNN
@@
 P 3120 1265
 F 0 "D1" H 3113 1481 50  0000 C CNN
-F 1 "LED" H 3113 1390 50  0000 C CNN
+F 1 "LED RED" H 3113 1390 50  0000 C CNN
 F 2 "LED_SMD:LED_1206_3216Metric" H 3120 1265 50  0001 C CNN
 F 3 "~" H 3120 1265 50  0001 C CNN
@@
 P 8450 1300
 F 0 "D5" H 8443 1516 50  0000 C CNN
-F 1 "LED" H 8443 1425 50  0000 C CNN
+F 1 "LED Yellow" H 8443 1425 50  0000 C CNN
 F 2 "LED_SMD:LED_1206_3216Metric" H 8450 1300 50  0001 C CNN
 F 3 "~" H 8450 1300 50  0001 C CNN
@@
 Wire Wire Line
 	4605 1305 4715 1305
+$Comp
+L Device:R R1
+U 1 1 5F1702EA
+P 3530 1265
+F 0 "R1" V 3323 1265 50  0000 C CNN
+F 1 "R" V 3414 1265 50  0000 C CNN
+F 2 "Resistor_SMD:R_0805_2012Metric_Pad1.15x1.40mm_HandSolder" V 3460 1265 50  0001 C CNN
+F 3 "~" H 3530 1265 50  0001 C CNN
+	1    3530 1265
+	0    1    1    0
+$EndComp
 $EndSCHEMATC
